File: Ultra_DB_X51_v1.kicad_pcb (KiCad board)
At the start: 2 copper layers, 178 x 145 mm, 141 parts, among them IC1 L293D, J1 USB_2, K1 RELAYPTH, K2 RELAYPTH, K3 I2C, K4 CONN_3, P1 CONN_5, P10 CONN_8, P11 CONN_4, P12 CONN_8, P13 CONN_1, P14 CONN_1, P15 CONN_1, P16 CONN_8, P17 CONN_8, P18 CONN_7, P19 CONN_1, P2 CONN_5, P3 CONN_5, P4 CONN_1, P5 CONN_5X2, P6 CONN_1, P7 CONN_8, P8 CONN_8, P9 CONN_8, Q1 BC557, Q2 BC548, Q3 BC548, Q4 BC548, Q5 BC548, Q6 BC548, Q7 BC548, Q8 BC548, SW1 SPST, SW10 5, SW11 6, SW12 7, SW13 8, SW14 1, SW15 2, SW16 3, SW17 4, SW18 SPST, SW19 INT0, SW2 C, SW20 INT1, SW3 D, SW4 E, SW5 F, SW6 9, SW7 0, SW8 A, SW9 B, U1 7805, U10 CP2102, U2 24C16, U3 DS1307, U4 BATTERY, U5 LM555N_XL, U6 ADC0808, U7 AT89S52, X1 CRYSTAL, X3 11.0592MHz

Commit message: Filled zones
Parts:
- added REF**: 1pin, Connect:1pin, F.Cu at (150.1, 35.0)
- added REF**: 1pin, Connect:1pin, F.Cu at (150.1, 66.0)
- added REF**: 1pin, Connect:1pin, F.Cu at (75.1, 35.0)
Routing:
- net GND: track 836.1 -> 842.2 mm
- net /Key Pad/OUT: track 25.5 -> 28.1 mm
- net +5V: track 907.7 -> 907.2 mm
- added copper zone on F.Cu, net +5V
- added copper zone on B.Cu, net GND
Other:
- board text added: "LCD POT"
