File: Ultra_DB_X51_v1.sch (KiCad schematic (older format))
At the start: 45 parts, among them J1 USB_2, K4 CONN_3, P1 CONN_5, P10 CONN_8, P14 CONN_1, P15 CONN_1, P19 CONN_1, P2 CONN_5, P3 CONN_5, P4 CONN_1, P5 CONN_5X2, P6 CONN_1, P7 CONN_8, P8 CONN_8, P9 CONN_8, Q1 BC557, SW1 SPST, SW18 SPST, SW19 INT0, SW20 INT1, U1 7805, U10 CP2102, U7 AT89S52, X3 11.0592MHz

Commit message: BOM
Parts:
- C1, C2: symbol CP1 -> CP1-RESCUE-Ultra_DB_X51_v1
- C11, C12, C7: symbol C -> C-RESCUE-Ultra_DB_X51_v1
- D15, D3: symbol LED -> LED-RESCUE-Ultra_DB_X51_v1
- R1, R10, R11, R12, R13, R17, R27: symbol R -> R-RESCUE-Ultra_DB_X51_v1
Changed lines of the file:
@@
 EESchema Schematic File Version 2
+LIBS:Ultra_DB_X51_v1-rescue
 LIBS:power
 LIBS:device
@@
 LIBS:memory
 LIBS:xilinx
-LIBS:special
 LIBS:microcontrollers
 LIBS:dsp
@@
 $EndComp
 $Comp
-L LED D3
+L LED-RESCUE-Ultra_DB_X51_v1 D3
 U 1 1 4FFCD3C4
 P 4000 6250
@@
 $EndComp
 $Comp
-L C C12
+L C-RESCUE-Ultra_DB_X51_v1 C12
 U 1 1 4FFCD3BE
 P 7800 3700
@@
 $EndComp
 $Comp
-L C C11
+L C-RESCUE-Ultra_DB_X51_v1 C11
 U 1 1 4FFCD3BD
 P 7200 3700
@@
 $EndComp
 $Comp
-L R R17
+L R-RESCUE-Ultra_DB_X51_v1 R17
 U 1 1 4FFCD3B5
 P 1950 3550
@@
 $EndComp
 $Comp
-L R R1
+L R-RESCUE-Ultra_DB_X51_v1 R1
 U 1 1 4FFCD3B4
 P 4000 5750
@@
 NoConn ~ 4900 3350
 $Comp
-L CP1 C2
+L CP1-RESCUE-Ultra_DB_X51_v1 C2
 U 1 1 4FFCD3A2
 P 5650 5950
@@
 $EndComp
 $Comp
-L CP1 C1
+L CP1-RESCUE-Ultra_DB_X51_v1 C1
 U 1 1 4FFCD39F
 P 4250 5900
@@
 $EndComp
 $Comp
-L C C7
+L C-RESCUE-Ultra_DB_X51_v1 C7
 U 1 1 548EB15B
 P 7550 5050
@@
 $EndComp
 $Comp
-L R R11
+L R-RESCUE-Ultra_DB_X51_v1 R11
 U 1 1 549512C0
 P 9350 3250
@@
 $EndComp
 $Comp
-L R R12
+L R-RESCUE-Ultra_DB_X51_v1 R12
 U 1 1 549512CD
 P 9650 3500
@@
 $EndComp
 $Comp
-L R R10
+L R-RESCUE-Ultra_DB_X51_v1 R10
 U 1 1 54951C2C
 P 9050 3500
@@
 Connection ~ 9650 3750
 $Comp
-L R R13
+L R-RESCUE-Ultra_DB_X51_v1 R13
 U 1 1 549521B7
 P 10350 3000
@@
 79 E3 73 01 AA 0D CF 9F 3C 98 C5 F6 CF AC 04 72 85 62 D7 80 77 B1 8B CB 18 6F AC E9 6A 17 BB B8
 C2 B0 6B C0 BB D8 C5 65 8C 5D 03 DE C5 2E 2E 63 EC 1A F0 2E 76 71 19 63 D7 80 77 B1 8B CB 18 BB
-06 BC 8B 5D 5C C6 F8 FF 01 52 B3 1C 8C A4 9D 25 1B 00 00 00 00 49 45 4E 44 AE 42 60 82 1B
+06 BC 8B 5D 5C C6 F8 FF 01 52 B3 1C 8C A4 9D 25 1B 00 00 00 00 49 45 4E 44 AE 42 60 82
 EndData
 $EndBitmap
@@
 Connection ~ 4200 2250
 $Comp
-L R R27
+L R-RESCUE-Ultra_DB_X51_v1 R27
 U 1 1 549E7B98
 P 10900 5400
@@
 $EndComp
 $Comp
-L LED D15
+L LED-RESCUE-Ultra_DB_X51_v1 D15
 U 1 1 549E7B9F
 P 10900 6000
